File: Main_Board/main_board.kicad_sch (KiCad schematic)
At the start: 15 parts, among them J1 MEGA_SARJ, J2 POWER, J3 I2C, J4 FREE_GPIO, J5 5V, J6 12V, J7 24V, J8 GND, J9 GND, U1 BNO055_IMU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

Commit message: all pcb design except routing completed.
Connections:
- net DCAN2RX: now also J4.4 (Pin_4)
- net DCAN2TX: now also J4.3 (Pin_3)
- net N2HET2_11: now also J4.2 (Pin_2)
- net N2HET2_13/MIBSPI2SOMI: now also U2.J10_46
- net N2HET2_23: now also J4.1 (Pin_1)
- net N2HET2_3/MIBSPI2CLK: now also J4.7 (Pin_7); no longer J4.1 (Pin_1)
- net N2HET2_4: now also J4.8 (Pin_8); no longer J4.2 (Pin_2)
- net N2HET2_9: now also MODULE1.5 (IN1)
- net AD2IN_23: now reaches J4.5 (Pin_5)
- net AD2IN_23: now also U2.J9_29
- net AD2IN_24: now reaches J4.6 (Pin_6)
- net AD2IN_24: now also U2.J9_30
- net +3V3: now reaches U2.J10_3
- net +3V3: now also U2.J9_3
Other:
- note removed: "TRANSIEVER_0 ile hem curtis hem bms can bağlantıları açıp kapatılacak. İleride istenirse ayrı ayrı yapabiliriz."
- moved on the sheet: J1, J3, U1, U3, U4

Commit message: pcb to completed gerber completed ready to print the PCB
Connections:
- net +3.3V: now also U2.J9_3
- net +3V3: no longer names the net of U2.J10_3
- net +3V3: no longer U2.J9_3
Changed lines of the file:
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@@
   (junction (at 218.44 74.93) (diameter 0) (color 0 0 0 0)
   )
+  (junction (at 71.755 131.445) (diameter 0) (color 0 0 0 0)
+  )
   (junction (at 218.44 65.405) (diameter 0) (color 0 0 0 0)
   )
@@
     (stroke (width 0) (type default) (color 0 0 0 0))
   )
-  (wire (pts (xy 158.115 106.045) (xy 165.1 106.045))
-    (stroke (width 0) (type default) (color 0 0 0 0))
-  )
   (wire (pts (xy 78.74 170.815) (xy 86.36 170.815))
     (stroke (width 0) (type default) (color 0 0 0 0))
@@
     (stroke (width 0) (type default) (color 0 0 0 0))
   )
-  (wire (pts (xy 78.74 131.445) (xy 86.36 131.445))
+  (wire (pts (xy 71.755 131.445) (xy 86.36 131.445))
     (stroke (width 0) (type default) (color 0 0 0 0))
   )
@@
   )
   (wire (pts (xy 218.44 62.865) (xy 218.44 65.405))
+    (stroke (width 0) (type default) (color 0 0 0 0))
+  )
+  (wire (pts (xy 67.945 131.445) (xy 71.755 131.445))
     (stroke (width 0) (type default) (color 0 0 0 0))
   )
@@
     (effects (font (size 0.889 0.889)) (justify left))
     (property "Intersheet References" "${INTERSHEET_REFS}" (id 0) (at 3.175 -22.225 0)
+      (effects (font (size 1.27 1.27)) hide)
+    )
+  )
+  (global_label "+3V3" (shape bidirectional) (at 67.945 131.445 180) (fields_autoplaced)
+    (effects (font (size 0.889 0.889)) (justify right))
+    (property "Intersheet References" "${INTERSHEET_REFS}" (id 0) (at 151.765 -247.015 0)
       (effects (font (size 1.27 1.27)) hide)
     )
@@
     (pin "1")
   )
-  (symbol (lib_id "power:+3.3V") (at 78.74 131.445 90) (unit 1)
-    (in_bom yes) (on_board yes)
-    (property "Reference" "#PWR0130" (id 0) (at 82.55 131.445 0)
-      (effects (font (size 1.27 1.27)) hide)
-    )
-    (property "Value" "+3.3V" (id 1) (at 69.85 131.445 90)
+  (symbol (lib_id "power:+3.3V") (at 71.755 131.445 0) (unit 1)
+    (in_bom yes) (on_board yes)
+    (property "Reference" "#PWR0130" (id 0) (at 71.755 135.255 0)
+      (effects (font (size 1.27 1.27)) hide)
+    )
+    (property "Value" "+3.3V" (id 1) (at 71.755 122.555 90)
       (effects (font (size 1.27 1.27)) (justify right))
     )
-    (property "Footprint" "" (id 2) (at 78.74 131.445 0)
-      (effects (font (size 1.27 1.27)) hide)
-    )
-    (property "Datasheet" "" (id 3) (at 78.74 131.445 0)
-      (effects (font (size 1.27 1.27)) hide)
-    )
+    (property "Footprint" "" (id 2) (at 71.755 131.445 0)
+      (effects (font (size 1.27 1.27)) hide)
+    )
+    (property "Datasheet" "" (id 3) (at 71.755 131.445 0)
+      (effects (font (size 1.27 1.27)) hide)
+    )
